File: Plant_Saver_Spring_2026/Plant_Saver_Kicad/TP4056_Solar.kicad_sch (KiCad schematic)
At the start: 6 parts, among them U7 TPB4056A20-ES1R

Commit message: Sensor Fun
Had to annotate in order to assign footprints, If that messed anything up I'd be happy to fix it. Added a basic 1x4 header for the temp sensor and added the correct female pins/header footprint for the capacitive moisture sensor. Also put a footprint in there for the OLED using the 4pin cable that we don't have but would be nice to. If we choose to go with the headers instead it's and easy change.
Parts:
- C10, C9: footprint CAP_C410C_AX_X7R_AXIMAX_KEM -> (none)
- U7: footprint ESOP-8_TPK -> (none)
Changed lines of the file:
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@@
 			)
 		)
-		(property "Footprint" "CAP_C410C_AX_X7R_AXIMAX_KEM"
+		(property "Footprint" ""
 			(at 204.1652 104.14 0)
 			(effects
@@
 			)
 		)
-		(property "Footprint" "ESOP-8_TPK"
+		(property "Footprint" ""
 			(at 128.27 91.44 0)
 			(effects
@@
 			)
 		)
-		(property "Footprint" "CAP_C410C_AX_X7R_AXIMAX_KEM"
+		(property "Footprint" ""
 			(at 127.9652 88.9 0)
 			(effects
