File: Plant_Saver_Spring_2026/Plant_Saver_Kicad/TP4056_USB.kicad_sch (KiCad schematic)
At the start: 6 parts, among them U8 TPB4056A20-ES1R

Commit message: Sensor Fun
Had to annotate in order to assign footprints, If that messed anything up I'd be happy to fix it. Added a basic 1x4 header for the temp sensor and added the correct female pins/header footprint for the capacitive moisture sensor. Also put a footprint in there for the OLED using the 4pin cable that we don't have but would be nice to. If we choose to go with the headers instead it's and easy change.
Parts:
- C11, C12: footprint CAP_C410C_AX_X7R_AXIMAX_KEM -> (none)
- U8: footprint ESOP-8_TPK -> (none)
Changed lines of the file:
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@@
 			)
 		)
-		(property "Footprint" "ESOP-8_TPK"
+		(property "Footprint" ""
 			(at 109.22 93.98 0)
 			(effects
@@
 			)
 		)
-		(property "Footprint" "CAP_C410C_AX_X7R_AXIMAX_KEM"
+		(property "Footprint" ""
 			(at 108.9152 91.44 0)
 			(effects
@@
 			)
 		)
-		(property "Footprint" "CAP_C410C_AX_X7R_AXIMAX_KEM"
+		(property "Footprint" ""
 			(at 185.1152 106.68 0)
 			(effects
