File: Plant_Saver_Spring_2026/Plant_Saver_Kicad/UVLO_Hysteresis.kicad_sch (KiCad schematic)
At the start: 8 parts, among them Q2 SSF1341, U9 MCP6546-I/P

Commit message: Sensor Fun
Had to annotate in order to assign footprints, If that messed anything up I'd be happy to fix it. Added a basic 1x4 header for the temp sensor and added the correct female pins/header footprint for the capacitive moisture sensor. Also put a footprint in there for the OLED using the 4pin cable that we don't have but would be nice to. If we choose to go with the headers instead it's and easy change.
Parts:
- U9: footprint PDIP8_300MC_MCH -> (none)
Changed lines of the file:
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@@
 			)
 		)
-		(property "Footprint" "PDIP8_300MC_MCH"
+		(property "Footprint" ""
 			(at 109.22 96.52 0)
 			(effects
