File: Plant_Saver_Spring_2026/Plant_Saver_Kicad/Solar_Measurement_Unit.kicad_sch (KiCad schematic)
At the start: 7 parts, among them U12 LM358AP

Commit message: Sensor Fun
Had to annotate in order to assign footprints, If that messed anything up I'd be happy to fix it. Added a basic 1x4 header for the temp sensor and added the correct female pins/header footprint for the capacitive moisture sensor. Also put a footprint in there for the OLED using the 4pin cable that we don't have but would be nice to. If we choose to go with the headers instead it's and easy change.
Parts:
- U12: footprint P8 -> (none)
Changed lines of the file:
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@@
 			)
 		)
-		(property "Footprint" "P8"
+		(property "Footprint" ""
 			(at 109.22 85.09 0)
 			(effects

Commit message: Updates to power schematic
Replaced certain selection transistors for lower Rds_on, added thermal cutoff and DW03 for battery protection, swapped in 4-channel op-amps for solar measurement, various misc. improvements.
Parts:
- renumbered R3 to R11, R4 to R12, R5 to R39, R6 to R40, R30 to R41, R31 to R42, U12 to U8
Changed lines of the file:
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@@
 		(dnp no)
 		(fields_autoplaced yes)
-		(property "Reference" "R30"
+		(property "Reference" "R41"
 			(at 179.07 95.2499 0)
 			(effects
@@
 				(path "/7f244634-d37a-4ff0-ba36-8027330ab1bd/6d8064f9-fe21-41d8-9d65-91dc024fa0a0"
 					(reference "R30")
+					(unit 1)
+				)
+				(path "/7f244634-d37a-4ff0-ba36-8027330ab1bd/f38af1ac-5094-49ba-9dea-0c29bb6881a5"
+					(reference "R41")
 					(unit 1)
 				)
@@
 		(dnp no)
 		(fields_autoplaced yes)
-		(property "Reference" "R6"
+		(property "Reference" "R40"
 			(at 139.7 64.77 90)
 			(effects
@@
 				(path "/7f244634-d37a-4ff0-ba36-8027330ab1bd/6d8064f9-fe21-41d8-9d65-91dc024fa0a0"
 					(reference "R6")
+					(unit 1)
+				)
+				(path "/7f244634-d37a-4ff0-ba36-8027330ab1bd/f38af1ac-5094-49ba-9dea-0c29bb6881a5"
+					(reference "R40")
 					(unit 1)
 				)
@@
 		(dnp no)
 		(fields_autoplaced yes)
-		(property "Reference" "U12"
+		(property "Reference" "U8"
 			(at 139.7 74.93 0)
 			(effects
@@
 				(path "/7f244634-d37a-4ff0-ba36-8027330ab1bd/6d8064f9-fe21-41d8-9d65-91dc024fa0a0"
 					(reference "U12")
+					(unit 1)
+				)
+				(path "/7f244634-d37a-4ff0-ba36-8027330ab1bd/f38af1ac-5094-49ba-9dea-0c29bb6881a5"
+					(reference "U8")
 					(unit 1)
 				)
@@
 		(dnp no)
 		(fields_autoplaced yes)
-		(property "Reference" "R3"
+		(property "Reference" "R11"
 			(at 91.44 81.28 90)
 			(effects
@@
 				(path "/7f244634-d37a-4ff0-ba36-8027330ab1bd/6d8064f9-fe21-41d8-9d65-91dc024fa0a0"
 					(reference "R3")
+					(unit 1)
+				)
+				(path "/7f244634-d37a-4ff0-ba36-8027330ab1bd/f38af1ac-5094-49ba-9dea-0c29bb6881a5"
+					(reference "R11")
 					(unit 1)
 				)
@@
 		(dnp no)
 		(fields_autoplaced yes)
-		(property "Reference" "R5"
+		(property "Reference" "R39"
 			(at 102.87 78.74 90)
 			(effects
@@
 				(path "/7f244634-d37a-4ff0-ba36-8027330ab1bd/6d8064f9-fe21-41d8-9d65-91dc024fa0a0"
 					(reference "R5")
+					(unit 1)
+				)
+				(path "/7f244634-d37a-4ff0-ba36-8027330ab1bd/f38af1ac-5094-49ba-9dea-0c29bb6881a5"
+					(reference "R39")
 					(unit 1)
 				)
@@
 		(dnp no)
 		(fields_autoplaced yes)
-		(property "Reference" "R31"
+		(property "Reference" "R42"
 			(at 195.58 81.28 90)
 			(effects
@@
 				(path "/7f244634-d37a-4ff0-ba36-8027330ab1bd/6d8064f9-fe21-41d8-9d65-91dc024fa0a0"
 					(reference "R31")
+					(unit 1)
+				)
+				(path "/7f244634-d37a-4ff0-ba36-8027330ab1bd/f38af1ac-5094-49ba-9dea-0c29bb6881a5"
+					(reference "R42")
 					(unit 1)
 				)
@@
 		(dnp no)
 		(fields_autoplaced yes)
-		(property "Reference" "R4"
+		(property "Reference" "R12"
 			(at 101.6 92.7099 0)
 			(effects
@@
 					(unit 1)
 				)
+				(path "/7f244634-d37a-4ff0-ba36-8027330ab1bd/f38af1ac-5094-49ba-9dea-0c29bb6881a5"
+					(reference "R12")
+					(unit 1)
+				)
