File: Plant_Saver_Spring_2026/Plant_Saver_Kicad/Linear_Regulator.kicad_sch (KiCad schematic)
At the start: 7 parts, among them U1 LP38511TJ-ADJ/NOPB

Commit message: Sensor Fun
Had to annotate in order to assign footprints, If that messed anything up I'd be happy to fix it. Added a basic 1x4 header for the temp sensor and added the correct female pins/header footprint for the capacitive moisture sensor. Also put a footprint in there for the OLED using the 4pin cable that we don't have but would be nice to. If we choose to go with the headers instead it's and easy change.
Parts:
- U1: footprint TJ5A_TEX -> (none)
Changed lines of the file:
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@@
 			)
 		)
-		(property "Footprint" "TJ5A_TEX"
+		(property "Footprint" ""
 			(at 71.12 66.04 0)
 			(effects

Commit message: Footprint correction
Changed the DHT20 from a header pin to the recommended SIP. Also had to reannotate in order to assign footprints.
Parts:
- removed C1, C2: 10uF, Capacitor_THT:C_Disc_D4.7mm_W2.5mm_P5.00mm, symbol Device:C
- removed C3: 1nF, Capacitor_THT:C_Disc_D3.8mm_W2.6mm_P2.50mm, symbol Device:C
- removed R2: 100K, Resistor_THT:R_Axial_DIN0207_L6.3mm_D2.5mm_P10.16mm_Horizontal, symbol Device:R_US
- removed R28: 5.6K, Resistor_THT:R_Axial_DIN0207_L6.3mm_D2.5mm_P10.16mm_Horizontal, symbol Device:R_US
- removed R29: 1K, Resistor_THT:R_Axial_DIN0207_L6.3mm_D2.5mm_P10.16mm_Horizontal, symbol Device:R_US
- removed U1: LP38511TJ-ADJ/NOPB, symbol LP38511TJ_ADJ_NOPB:LP38511TJ-ADJ_NOPB

Commit message: Fixed USB-C and Linear Regulator Sheetfiles
Parts:
- added C1, C2: 10uF, Capacitor_THT:C_Disc_D4.7mm_W2.5mm_P5.00mm, symbol Device:C
- added C3: 1nF, Capacitor_THT:C_Disc_D3.8mm_W2.6mm_P2.50mm, symbol Device:C
- added R2: 100K, Resistor_THT:R_Axial_DIN0207_L6.3mm_D2.5mm_P10.16mm_Horizontal, symbol Device:R_US
- added R28: 5.6K, Resistor_THT:R_Axial_DIN0207_L6.3mm_D2.5mm_P10.16mm_Horizontal, symbol Device:R_US
- added R29: 1K, Resistor_THT:R_Axial_DIN0207_L6.3mm_D2.5mm_P10.16mm_Horizontal, symbol Device:R_US
- added U1: LP38511TJ-ADJ/NOPB, symbol LP38511TJ_ADJ_NOPB:LP38511TJ-ADJ_NOPB
Connections:
- new net: C3.1, R28.1, R29.2, U1.5 (ADJ)
- new net: R2.1, U1.1 (EN)
- new net GND: C1.2, C2.2, R29.1, U1.3 (GND), U1.6 (DAP)
- new net Vin: C1.1, R2.2, U1.2 (IN)
- new net Vout: C2.1, C3.2, R28.2, U1.4 (OUT)

Commit message: Started PCB
Parts:
- U12: renamed from U1; footprint (none) -> LP38511TJ_ADJ_NOPB:TJ5A_TEX
- renumbered C1 to C6, C2 to C7, C3 to C8, R2 to R15, R29 to R16, R28 to R17
Changed lines of the file:
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@@
 		(on_board yes)
 		(dnp no)
-		(property "Reference" "C2"
+		(property "Reference" "C7"
 			(at 156.972 99.06 0)
 			(effects
@@
 			(project "Plant_Saver_Dev"
 				(path "/7f244634-d37a-4ff0-ba36-8027330ab1bd/c1b5c94f-5fb5-4e2b-895b-5d171c372d7d/a8348cc8-6eff-45be-a6d2-3e9c25423c18"
-					(reference "C2")
+					(reference "C7")
 					(unit 1)
 				)
@@
 		(dnp no)
 		(fields_autoplaced yes)
-		(property "Reference" "#PWR017"
+		(property "Reference" "#PWR025"
 			(at 119.38 110.49 0)
 			(effects
@@
 			(project "Plant_Saver_Dev"
 				(path "/7f244634-d37a-4ff0-ba36-8027330ab1bd/c1b5c94f-5fb5-4e2b-895b-5d171c372d7d/a8348cc8-6eff-45be-a6d2-3e9c25423c18"
-					(reference "#PWR017")
+					(reference "#PWR025")
 					(unit 1)
 				)
@@
 		(dnp no)
 		(fields_autoplaced yes)
-		(property "Reference" "C1"
+		(property "Reference" "C6"
 			(at 81.28 91.4399 0)
 			(effects
@@
 			(project "Plant_Saver_Dev"
 				(path "/7f244634-d37a-4ff0-ba36-8027330ab1bd/c1b5c94f-5fb5-4e2b-895b-5d171c372d7d/a8348cc8-6eff-45be-a6d2-3e9c25423c18"
-					(reference "C1")
+					(reference "C6")
 					(unit 1)
 				)
@@
 		(dnp no)
 		(fields_autoplaced yes)
-		(property "Reference" "R29"
+		(property "Reference" "R16"
 			(at 156.21 83.8199 0)
 			(effects
@@
 			(project "Plant_Saver_Dev"
 				(path "/7f244634-d37a-4ff0-ba36-8027330ab1bd/c1b5c94f-5fb5-4e2b-895b-5d171c372d7d/a8348cc8-6eff-45be-a6d2-3e9c25423c18"
-					(reference "R29")
+					(reference "R16")
 					(unit 1)
 				)
@@
 		(dnp no)
 		(fields_autoplaced yes)
-		(property "Reference" "R2"
+		(property "Reference" "R15"
 			(at 85.09 83.8199 0)
 			(effects
@@
 			(project "Plant_Saver_Dev"
 				(path "/7f244634-d37a-4ff0-ba36-8027330ab1bd/c1b5c94f-5fb5-4e2b-895b-5d171c372d7d/a8348cc8-6eff-45be-a6d2-3e9c25423c18"
-					(reference "R2")
+					(reference "R15")
 					(unit 1)
 				)
@@
 		(dnp no)
 		(fields_autoplaced yes)
-		(property "Reference" "U1"
+		(property "Reference" "U12"
 			(at 119.38 81.28 0)
 			(effects
@@
 			)
 		)
-		(property "Footprint" ""
+		(property "Footprint" "LP38511TJ_ADJ_NOPB:TJ5A_TEX"
 			(at 91.44 91.44 0)
 			(effects
@@
 			(project ""
 				(path "/7f244634-d37a-4ff0-ba36-8027330ab1bd/c1b5c94f-5fb5-4e2b-895b-5d171c372d7d/a8348cc8-6eff-45be-a6d2-3e9c25423c18"
-					(reference "U1")
+					(reference "U12")
 					(unit 1)
 				)
@@
 		(on_board yes)
 		(dnp no)
-		(property "Reference" "C3"
+		(property "Reference" "C8"
 			(at 168.402 91.44 0)
 			(effects
@@
 			(project "Plant_Saver_Dev"
 				(path "/7f244634-d37a-4ff0-ba36-8027330ab1bd/c1b5c94f-5fb5-4e2b-895b-5d171c372d7d/a8348cc8-6eff-45be-a6d2-3e9c25423c18"
-					(reference "C3")
+					(reference "C8")
 					(unit 1)
 				)
@@
 		(dnp no)
 		(fields_autoplaced yes)
-		(property "Reference" "R28"
+		(property "Reference" "R17"
 			(at 156.21 91.4399 0)
 			(effects
@@
 			(project "Plant_Saver_Dev"
 				(path "/7f244634-d37a-4ff0-ba36-8027330ab1bd/c1b5c94f-5fb5-4e2b-895b-5d171c372d7d/a8348cc8-6eff-45be-a6d2-3e9c25423c18"
-					(reference "R28")
+					(reference "R17")
 					(unit 1)
 				)
@@
 		(dnp no)
 		(fields_autoplaced yes)
-		(property "Reference" "#PWR018"
+		(property "Reference" "#PWR026"
 			(at 170.18 87.63 0)
 			(effects
@@
 			(project "Plant_Saver_Dev"
 				(path "/7f244634-d37a-4ff0-ba36-8027330ab1bd/c1b5c94f-5fb5-4e2b-895b-5d171c372d7d/a8348cc8-6eff-45be-a6d2-3e9c25423c18"
-					(reference "#PWR018")
-					(unit 1)
-				)
+					(reference "#PWR026")
+					(unit 1)
+				)

Commit message: Refined PCB layout
Parts:
- C6, C7: footprint Capacitor_THT:C_Disc_D4.7mm_W2.5mm_P5.00mm -> Capacitor_SMD:C_1206_3216Metric_Pad1.33x1.80mm_HandSolder
- C8: footprint Capacitor_THT:C_Disc_D3.8mm_W2.6mm_P2.50mm -> Capacitor_SMD:C_1206_3216Metric_Pad1.33x1.80mm_HandSolder
- R15: footprint Resistor_THT:R_Axial_DIN0207_L6.3mm_D2.5mm_P10.16mm_Horizontal -> Resistor_SMD:R_1206_3216Metric_Pad1.30x1.75mm_HandSolder
Changed lines of the file:
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@@
+	(wire
+		(pts
+			(xy 119.38 107.95) (xy 119.38 104.14)
+		)
+		(stroke
+			(width 0)
+			(type default)
+		)
+	)
 	(wire
 		(pts
@@
 			)
 		)
-		(property "Footprint" "Capacitor_THT:C_Disc_D4.7mm_W2.5mm_P5.00mm"
+		(property "Footprint" "Capacitor_SMD:C_1206_3216Metric_Pad1.33x1.80mm_HandSolder"
 			(at 154.6352 104.14 0)
 			(effects
@@
 	(symbol
 		(lib_id "power:GND")
-		(at 119.38 104.14 0)
+		(at 119.38 107.95 0)
 		(unit 1)
 		(exclude_from_sim no)
@@
 		(fields_autoplaced yes)
 		(property "Reference" "#PWR025"
-			(at 119.38 110.49 0)
+			(at 119.38 114.3 0)
 			(effects
 				(font
@@
 		)
 		(property "Value" "GND"
-			(at 119.38 109.22 0)
+			(at 119.38 113.03 0)
 			(effects
 				(font
@@
 		)
 		(property "Footprint" ""
-			(at 119.38 104.14 0)
+			(at 119.38 107.95 0)
 			(effects
 				(font
@@
 		)
 		(property "Datasheet" ""
-			(at 119.38 104.14 0)
+			(at 119.38 107.95 0)
 			(effects
 				(font
@@
 		)
 		(property "Description" "Power symbol creates a global label with name \"GND\" , ground"
-			(at 119.38 104.14 0)
+			(at 119.38 107.95 0)
 			(effects
 				(font
@@
 			)
 		)
-		(property "Footprint" "Capacitor_THT:C_Disc_D4.7mm_W2.5mm_P5.00mm"
+		(property "Footprint" "Capacitor_SMD:C_1206_3216Metric_Pad1.33x1.80mm_HandSolder"
 			(at 78.4352 96.52 0)
 			(effects
@@
 			)
 		)
-		(property "Footprint" "Resistor_THT:R_Axial_DIN0207_L6.3mm_D2.5mm_P10.16mm_Horizontal"
+		(property "Footprint" "Resistor_SMD:R_1206_3216Metric_Pad1.30x1.75mm_HandSolder"
 			(at 83.566 85.344 90)
 			(effects
@@
 			)
 		)
-		(property "Footprint" "Capacitor_THT:C_Disc_D3.8mm_W2.6mm_P2.50mm"
+		(property "Footprint" "Capacitor_SMD:C_1206_3216Metric_Pad1.33x1.80mm_HandSolder"
 			(at 166.0652 96.52 0)
 			(effects

Commit message: PCB Pre-Check complete
Parts:
- renumbered R15 to R16, R16 to R17, R17 to R18
Changed lines of the file:
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@@
 		(dnp no)
 		(fields_autoplaced yes)
-		(property "Reference" "R16"
+		(property "Reference" "R17"
 			(at 156.21 83.8199 0)
 			(effects
@@
 			(project "Plant_Saver_Dev"
 				(path "/7f244634-d37a-4ff0-ba36-8027330ab1bd/c1b5c94f-5fb5-4e2b-895b-5d171c372d7d/a8348cc8-6eff-45be-a6d2-3e9c25423c18"
-					(reference "R16")
+					(reference "R17")
 					(unit 1)
 				)
@@
 		(dnp no)
 		(fields_autoplaced yes)
-		(property "Reference" "R15"
+		(property "Reference" "R16"
 			(at 85.09 83.8199 0)
 			(effects
@@
 			(project "Plant_Saver_Dev"
 				(path "/7f244634-d37a-4ff0-ba36-8027330ab1bd/c1b5c94f-5fb5-4e2b-895b-5d171c372d7d/a8348cc8-6eff-45be-a6d2-3e9c25423c18"
-					(reference "R15")
+					(reference "R16")
 					(unit 1)
 				)
@@
 		(dnp no)
 		(fields_autoplaced yes)
-		(property "Reference" "R17"
+		(property "Reference" "R18"
 			(at 156.21 91.4399 0)
 			(effects
@@
 			(project "Plant_Saver_Dev"
 				(path "/7f244634-d37a-4ff0-ba36-8027330ab1bd/c1b5c94f-5fb5-4e2b-895b-5d171c372d7d/a8348cc8-6eff-45be-a6d2-3e9c25423c18"
-					(reference "R17")
-					(unit 1)
-				)
+					(reference "R18")
+					(unit 1)
+				)
