File: Plant_Saver_Spring_2026/Plant_Saver_Kicad/UOVLO_Solar.kicad_sch (KiCad schematic)
At the start: 11 parts, among them Q11 ISP12DP06NMXTSA1, Q12 G09P02L, U16 MCP6547T_I_MS

Commit message: PCB Pre-Check complete
Parts:
- renumbered R37 to R39, R38 to R40, R39 to R41, R40 to R42, R41 to R43, R42 to R44, R43 to R45
Changed lines of the file:
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@@
 		(dnp no)
 		(fields_autoplaced yes)
-		(property "Reference" "R38"
+		(property "Reference" "R40"
 			(at 116.84 91.4399 0)
 			(effects
@@
 			(project "Plant_Saver_Dev"
 				(path "/7f244634-d37a-4ff0-ba36-8027330ab1bd/c1b5c94f-5fb5-4e2b-895b-5d171c372d7d/9fa29de7-25a7-4316-bbea-8ab2651dedf4"
-					(reference "R38")
+					(reference "R40")
 					(unit 1)
 				)
@@
 		(dnp no)
 		(fields_autoplaced yes)
-		(property "Reference" "R40"
+		(property "Reference" "R42"
 			(at 140.97 83.8199 0)
 			(effects
@@
 			(project "Plant_Saver_Dev"
 				(path "/7f244634-d37a-4ff0-ba36-8027330ab1bd/c1b5c94f-5fb5-4e2b-895b-5d171c372d7d/9fa29de7-25a7-4316-bbea-8ab2651dedf4"
-					(reference "R40")
+					(reference "R42")
 					(unit 1)
 				)
@@
 		(dnp no)
 		(fields_autoplaced yes)
-		(property "Reference" "R43"
+		(property "Reference" "R45"
 			(at 203.2 74.93 90)
 			(effects
@@
 			(project "Plant_Saver_Dev"
 				(path "/7f244634-d37a-4ff0-ba36-8027330ab1bd/c1b5c94f-5fb5-4e2b-895b-5d171c372d7d/9fa29de7-25a7-4316-bbea-8ab2651dedf4"
-					(reference "R43")
+					(reference "R45")
 					(unit 1)
 				)
@@
 		(dnp no)
 		(fields_autoplaced yes)
-		(property "Reference" "R39"
+		(property "Reference" "R41"
 			(at 116.84 110.4899 0)
 			(effects
@@
 			(project "Plant_Saver_Dev"
 				(path "/7f244634-d37a-4ff0-ba36-8027330ab1bd/c1b5c94f-5fb5-4e2b-895b-5d171c372d7d/9fa29de7-25a7-4316-bbea-8ab2651dedf4"
-					(reference "R39")
+					(reference "R41")
 					(unit 1)
 				)
@@
 		(dnp no)
 		(fields_autoplaced yes)
-		(property "Reference" "R42"
+		(property "Reference" "R44"
 			(at 175.26 73.6599 0)
 			(effects
@@
 			(project "Plant_Saver_Dev"
 				(path "/7f244634-d37a-4ff0-ba36-8027330ab1bd/c1b5c94f-5fb5-4e2b-895b-5d171c372d7d/9fa29de7-25a7-4316-bbea-8ab2651dedf4"
-					(reference "R42")
+					(reference "R44")
 					(unit 1)
 				)
@@
 		(dnp no)
 		(fields_autoplaced yes)
-		(property "Reference" "R37"
+		(property "Reference" "R39"
 			(at 116.84 73.6599 0)
 			(effects
@@
 			(project "Plant_Saver_Dev"
 				(path "/7f244634-d37a-4ff0-ba36-8027330ab1bd/c1b5c94f-5fb5-4e2b-895b-5d171c372d7d/9fa29de7-25a7-4316-bbea-8ab2651dedf4"
-					(reference "R37")
+					(reference "R39")
 					(unit 1)
 				)
@@
 		(dnp no)
 		(fields_autoplaced yes)
-		(property "Reference" "R41"
+		(property "Reference" "R43"
 			(at 140.97 96.5199 0)
 			(effects
@@
 			(project "Plant_Saver_Dev"
 				(path "/7f244634-d37a-4ff0-ba36-8027330ab1bd/c1b5c94f-5fb5-4e2b-895b-5d171c372d7d/9fa29de7-25a7-4316-bbea-8ab2651dedf4"
-					(reference "R41")
-					(unit 1)
-				)
+					(reference "R43")
+					(unit 1)
+				)
