File: Plant_Saver_Spring_2026/Plant_Saver_Kicad/Charge_Circuit.kicad_sch (KiCad schematic)
At the start: 25 parts, among them J10 1.25mm, Q10 G09P02L, Q3 ISP12DP06NMXTSA1, Q4 G09P02L, Q5 G09P02L, Q6 G09P02L, Q7 G09P02L, Q8 G09P02L, Q9 G09P02L, SW4 SA72SB0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

Commit message: PCB Finishing Steps
Added additional details on silkscreen, added ground plane, misc. touchups
Parts:
- renumbered BUS1 to Bus1
Changed lines of the file:
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@@
 		(on_board yes)
 		(dnp no)
-		(fields_autoplaced yes)
 		(property "Reference" "BAT1"
-			(at 184.15 94.7419 0)
+			(at 184.15 94.742 0)
 			(effects
 				(font
@@
 		(dnp no)
 		(fields_autoplaced yes)
-		(property "Reference" "BUS1"
+		(property "Reference" "Bus1"
 			(at 270.51 99.8219 0)
 			(effects
@@
 			(project "Plant_Saver_Kicad"
 				(path "/7f244634-d37a-4ff0-ba36-8027330ab1bd/c1b5c94f-5fb5-4e2b-895b-5d171c372d7d"
-					(reference "BUS1")
-					(unit 1)
-				)
+					(reference "Bus1")
+					(unit 1)
+				)
