File: Plant_Saver_Spring_2026/Plant_Saver_Kicad/Plant_Saver_Kicad.kicad_pcb (KiCad board)
At the start: 2 copper layers, 82 x 85 mm, 114 parts, among them J10 1.25mm, J11 DM3D-SF, J2 SBH11-PBPC-D05-ST-BK, J3 Test, J4 SM04B-SRSS-TB, J6 Conn_01x02_Pin, J7 Conn_01x06_Socket, J8 S3B-PH-K-S, J9 54-00284, Q1 G09P02L, Q10 G09P02L, Q11 ISP12DP06NMXTSA1, Q12 G09P02L, Q2 G09P02L, Q3 ISP12DP06NMXTSA1, Q4 G09P02L, Q5 G09P02L, Q6 G09P02L, Q7 G09P02L, Q8 G09P02L, Q9 G09P02L, SW2 1101M2S3AQE2, SW4 SA72SB0, U1 CDBA140SL-HF, U10 DW03C, U11 CDBA140SL-HF, U12 LP38511TJ-ADJ/NOPB, U13 MCP73833-xxx-UN, U14 MCP6234, U15 MCP73833-xxx-UN, U16 MCP6547T_I_MS, U2 CDBA140SL-HF, U3 CDBA140SL-HF, U4 CDBA140SL-HF, U5 ESP32-WROOM-32E-N16, U9 CDBA140SL-HF

Commit message: Quick clearance adjustment on PCB
Parts:
- moved R4 14.0 mm to (131.5, 116.2), turned to -90 degrees
Routing:
- net Net-(U5-IO2): track 6.38 -> 21.3 mm
- net Vbus: track 183.6 -> 186.5 mm
- net GND: track 318.9 -> 317.3 mm
Changed lines of the file:
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@@
 	(footprint "Resistor_SMD:R_1206_3216Metric_Pad1.30x1.75mm_HandSolder"
 		(layer "F.Cu")
-		(at 145.5 116.2 90)
+		(at 131.5 116.2 -90)
 		(descr "Resistor SMD 1206 (3216 Metric), square (rectangular) end terminal, IPC-7351 nominal with elongated pad for handsoldering. (Body size source: IPC-SM-782 page 72, https://www.pcb-3d.com/wordpress/wp-content/uploads/ipc-sm-782a_amendment_1_and_2.pdf), generated with kicad-footprint-generator")
 		(tags "resistor handsolder")
@@
 		(attr smd)
 		(fp_line
-			(start -0.727064 -0.91)
-			(end 0.727064 -0.91)
+			(start -0.727064 0.91)
+			(end 0.727064 0.91)
 			(stroke
 				(width 0.12)
@@
 		)
 		(fp_line
-			(start -0.727064 0.91)
-			(end 0.727064 0.91)
+			(start -0.727064 -0.91)
+			(end 0.727064 -0.91)
 			(stroke
 				(width 0.12)
@@
 		)
 		(pad "1" smd roundrect
-			(at -1.55 0 90)
+			(at -1.55 0 270)
 			(size 1.3 1.75)
 			(layers "F.Cu" "F.Mask" "F.Paste")
@@
 		)
 		(pad "2" smd roundrect
-			(at 1.55 0 90)
+			(at 1.55 0 270)
 			(size 1.3 1.75)
 			(layers "F.Cu" "F.Mask" "F.Paste")
@@
 	)
 	(segment
-		(start 133.3 121.8)
-		(end 129.7063 118.2063)
-		(width 0.4)
-		(layer "F.Cu")
-		(net 1)
-	)
-	(segment
 		(start 133.1 85.5)
 		(end 133.1 93.40926)
@@
 	)
 	(segment
-		(start 153.126871 113.973129)
-		(end 145.3 121.8)
+		(start 125.35 114.75)
+		(end 132.4 121.8)
 		(width 0.4)
 		(layer "F.Cu")
@@
 	)
 	(segment
-		(start 153.128285 113.973129)
-		(end 153.126871 113.973129)
-		(width 0.4)
-		(layer "F.Cu")
-		(net 1)
-	)
-	(segment
 		(start 140.174999 65.361998)
 		(end 140.174999 67.083521)
@@
 	)
 	(segment
-		(start 135.4 112)
-		(end 132.4563 112)
+		(start 178.29 117.81)
+		(end 176.6 119.5)
 		(width 0.4)
 		(layer "F.Cu")
@@
 	)
 	(segment
-		(start 178.29 117.81)
-		(end 176.6 119.5)
+		(start 132.4 121.8)
+		(end 145.3 121.8)
 		(width 0.4)
 		(layer "F.Cu")
@@
 	)
 	(segment
+		(start 135.4 112)
+		(end 127.54506 112)
+		(width 0.4)
+		(layer "F.Cu")
+		(net 1)
+	)
+	(segment
 		(start 136.949 110.451)
 		(end 135.4 112)
@@
 	)
 	(segment
-		(start 171.1 126)
-		(end 171.1 129.632301)
+		(start 145.3 121.8)
+		(end 153.126871 113.973129)
 		(width 0.4)
 		(layer "F.Cu")
@@
 	)
 	(segment
-		(start 129.7063 114.75)
-		(end 130.87815 113.57815)
+		(start 124.79506 114.75)
+		(end 123.85 114.75)
 		(width 0.4)
 		(layer "F.Cu")
@@
 	)
 	(segment
-		(start 136.6125 81.5625)
-		(end 136.6 81.55)
+		(start 171.1 126)
+		(end 171.1 129.632301)
+		(width 0.4)
+		(layer "F.Cu")
+		(net 1)
+	)
+	(segment
+		(start 124.79506 114.75)
+		(end 125.35 114.75)
 		(width 0.4)
 		(layer "F.Cu")
@@
 	)
 	(segment
-		(start 123.85 114.75)
-		(end 129.7063 114.75)
+		(start 136.6125 81.5625)
+		(end 136.6 81.55)
 		(width 0.4)
 		(layer "F.Cu")
@@
 	)
 	(segment
-		(start 129.7063 118.2063)
-		(end 129.7063 114.75)
-		(width 0.4)
-		(layer "F.Cu")
-		(net 1)
-	)
-	(segment
 		(start 140.6 72.0625)
 		(end 139.1 70.5625)
@@
 	)
 	(segment
-		(start 145.3 121.8)
-		(end 133.3 121.8)
-		(width 0.4)
-		(layer "F.Cu")
-		(net 1)
-	)
-	(segment
 		(start 136.949 95.38316)
 		(end 136.949 110.451)
@@
 	)
 	(segment
-		(start 134.2004 94.50966)
-		(end 135.3497 94.50966)
+		(start 127.54506 112)
+		(end 124.79506 114.75)
 		(width 0.4)
 		(layer "F.Cu")
@@
 	)
 	(segment
-		(start 132.4563 112)
-		(end 130.87815 113.57815)
+		(start 134.2004 94.50966)
+		(end 135.3497 94.50966)
 		(width 0.4)
 		(layer "F.Cu")
@@
 	)
 	(segment
+		(start 153.126871 113.973129)
+		(end 153.128285 113.973129)
+		(width 0.4)
+		(layer "F.Cu")
+		(net 1)
+	)
+	(segment
 		(start 139.1 81.5625)
 		(end 136.6125 81.5625)
@@
 	)
 	(segment
+		(start 132.1 115.25)
+		(end 131.5 114.65)
+		(width 0.2)
+		(layer "F.Cu")
+		(net 2)
+	)
+	(segment
 		(start 114.2725 129.319)
 		(end 114.2725 126.906)
@@
 	)
 	(segment
-		(start 143.85 117.75)
-		(end 141.35 115.25)
-		(width 0.2)
-		(layer "F.Cu")
-		(net 2)
-	)
-	(segment
 		(start 166.7 117.3375)
 		(end 166.7 119)
@@
 	)
 	(segment
-		(start 145.5 117.75)
-		(end 143.85 117.75)
-		(width 0.2)
-		(layer "F.Cu")
-		(net 2)
-	)
-	(segment
 		(start 157.1 70.75)
 		(end 157.1 68.4)
@@
 	)
 	(segment
+		(start 134.85 115.25)
+		(end 132.1 115.25)
+		(width 0.2)
+		(layer "F.Cu")
+		(net 2)
+	)
+	(segment
 		(start 181.1 93.5)
 		(end 182.1 93.5)
@@
 	)
 	(segment
-		(start 149.815 111.94991)
-		(end 149.815 111.00061)
+		(start 131.5 117.75)
+		(end 143.37041 117.75)
 		(width 0.2)
 		(layer "F.Cu")
@@
 	)
 	(segment
-		(start 147.11491 114.65)
-		(end 149.815 111.94991)
+		(start 149.815 111.30541)
+		(end 149.815 111.00061)
 		(width 0.2)
 		(layer "F.Cu")
@@
 	)
 	(segment
-		(start 145.5 114.65)
-		(end 147.11491 114.65)
+		(start 143.37041 117.75)
+		(end 149.815 111.30541)
 		(width 0.2)
 		(layer "F.Cu")
