File: Plant_Saver_Spring_2026/Plant_Saver_Kicad_V2/InterfaceStripboard.kicad_sch (KiCad schematic)
At the start: 10 parts, among them SW5 3-1825910-5, SW6 3-1825910-5, SW7 3-1825910-5, SW8 3-1825910-5

Commit message: Organized Repo
Connections:
- net 3V3 renamed USB
Changed lines of the file:
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@@
 	(text "**NOTE**\nCurrent-limiting resistor values may vary\ndepending on individual LED characteristics."
 		(exclude_from_sim no)
-		(at 149.606 48.514 0)
+		(at 149.86 47.498 0)
 		(effects
 			(font
@@
 		)
 	)
-	(hierarchical_label "3V3"
+	(hierarchical_label "USB"
 		(shape input)
 		(at 127 60.96 180)
