File: Plant_Saver_Spring_2026/Plant_Saver_Kicad_V2/Plant_Saver_Kicad_V2.kicad_pcb (KiCad board)
At the start: 2 copper layers, 82 x 85 mm, 115 parts, among them J10 1.25mm, J11 DM3D-SF, J2 SBH11-PBPC-D05-ST-BK, J3 Test, J4 SM04B-SRSS-TB, J6 Conn_01x02_Pin, J7 Conn_01x06_Socket, J8 S3B-PH-K-S, J9 54-00284, Q1 G09P02L, Q10 G09P02L, Q11 ISP12DP06NMXTSA1, Q12 G09P02L, Q2 G09P02L, Q3 ISP12DP06NMXTSA1, Q4 G09P02L, Q5 G09P02L, Q6 G09P02L, Q7 G09P02L, Q8 G09P02L, Q9 G09P02L, SW2 1101M2S3AQE2, SW4 SA72SB0, U1 CDBA140SL-HF, U10 DW03C, U11 CDBA140SL-HF, U12 LP38511TJ-ADJ/NOPB, U13 MCP73833-xxx-UN, U14 MCP6234, U15 MCP73833-xxx-UN, U16 MCP6547T_I_MS, U17 LM66100DCK, U2 CDBA140SL-HF, U3 CDBA140SL-HF, U4 CDBA140SL-HF, U5 ESP32-WROOM-32E-N16, U9 CDBA140SL-HF

Commit message: Organized Repo
Parts:
- removed C6, C7: 10uF, Capacitor_SMD:C_1206_3216Metric_Pad1.33x1.80mm_HandSolder
- removed C8: 1nF, Capacitor_SMD:C_1206_3216Metric_Pad1.33x1.80mm_HandSolder
- removed J3: Test, Connector_PinHeader_2.54mm:PinHeader_1x02_P2.54mm_Vertical
- removed R16: 100K, Resistor_SMD:R_1206_3216Metric_Pad1.30x1.75mm_HandSolder
- removed R17: 1K, Resistor_THT:R_Axial_DIN0207_L6.3mm_D2.5mm_P10.16mm_Horizontal
- removed R18: 5.6K, Resistor_THT:R_Axial_DIN0207_L6.3mm_D2.5mm_P10.16mm_Horizontal
- removed U12: LP38511TJ-ADJ/NOPB, LP38511TJ_ADJ_NOPB:TJ5A_TEX
- added C17: 1uF, Capacitor_SMD:C_1206_3216Metric_Pad1.33x1.80mm_HandSolder, F.Cu at (169.5, 100.3)
- added C18: 1uF, Capacitor_SMD:C_1206_3216Metric_Pad1.33x1.80mm_HandSolder, F.Cu at (165.1, 104.5)
- added U18: XC6210A332PR-G, Package_TO_SOT_SMD:SOT-89-5_Handsoldering, F.Cu at (169.4, 105.9)
- U11, U9: value CDBA140SL-HF -> VS_10BQ015HM3_5BT; footprint CDBA140SL_HF:CDBA-HF -> VS_10BQ015HM3_5BT:CR_SMBDO-214AA_VIS
- moved R2 6.69 mm to (172.1, 114.8), turned to 90 degrees
- moved Bus1 2.65 mm to (179.2, 108.8)
- moved U9 1.76 mm to (158.8, 93.1)
- moved U11 1.63 mm to (166.4, 93.1)
Connections:
- Bus1 pad 1: /Power_And_Charging/Vout -> Vbus
- J2 pad 1: Vbus -> /Power_And_Charging/Vbus_USB
- SW2 pad 1: Vbus -> Net-(SW2-B)
- SW2 pad 3: /Power_And_Charging/Vout -> /Power_And_Charging/Linear_Regulator/Vin
Routing:
- net /Power_And_Charging/Vout: track 78.6 -> 0.00 mm
- net /Power_And_Charging/Vbus_USB: track 66.9 -> 126.4 mm, vias 0 -> 1
- net Net-(SW2-B): track 0.00 -> 25.6 mm
- net GND: track 326.0 -> 302.9 mm, vias 6 -> 7
- net Net-(U12-ADJ): track 18.6 -> 0.00 mm
- net Error: track 52.6 -> 44.5 mm
- net Periph_EN: track 36.6 -> 29.2 mm
- net Vbus: track 174.6 -> 179.9 mm, vias 4 -> 5
- net Net-(U12-EN): track 3.72 -> 0.00 mm
- net Net-(Q10-G): track 31.3 -> 29.0 mm
- net /Power_And_Charging/Linear_Regulator/Vin: track 47.5 -> 49.1 mm
Other:
- board text removed: "Imeas"
