File: Plant_Saver_Spring_2026/Plant_Saver_Kicad_V2/Charge_Circuit.kicad_sch (KiCad schematic)
At the start: 25 parts, among them J10 1.25mm, Q10 G09P02L, Q3 ISP12DP06NMXTSA1, Q4 G09P02L, Q5 G09P02L, Q6 G09P02L, Q7 G09P02L, Q8 G09P02L, Q9 G09P02L, SW4 SA72SB0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

Commit message: Organized Repo
Parts:
- U11, U9: value CDBA140SL-HF -> VS_10BQ015HM3_5BT; footprint CDBA140SL_HF:CDBA-HF -> VS_10BQ015HM3_5BT:CR_SMBDO-214AA_VIS
Other:
- moved on the sheet: BAT1, BT1, Bus1, C5, J10, Q10, Q3, Q4, Q5, Q6, Q7, Q8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

Commit message: Added assets for readme
Other:
- moved on the sheet: SOLB1
Changed lines of the file:
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@@
 	)
 	(junction
-		(at 99.06 48.26)
+		(at 97.79 48.26)
 		(diameter 0)
 		(color 0 0 0 0)
@@
 	)
 	(junction
-		(at 100.33 48.26)
-		(diameter 0)
-		(color 0 0 0 0)
-	)
-	(junction
 		(at 72.39 48.26)
 		(diameter 0)
@@
 	)
 	(junction
+		(at 97.79 38.1)
+		(diameter 0)
+		(color 0 0 0 0)
+	)
+	(junction
 		(at 191.77 119.38)
 		(diameter 0)
@@
 	(wire
 		(pts
-			(xy 99.06 48.26) (xy 100.33 48.26)
-		)
-		(stroke
-			(width 0)
-			(type default)
-		)
-	)
-	(wire
-		(pts
 			(xy 85.09 55.88) (xy 81.28 55.88)
 		)
@@
 	(wire
 		(pts
-			(xy 100.33 48.26) (xy 100.33 66.04)
-		)
-		(stroke
-			(width 0)
-			(type default)
-		)
-	)
-	(wire
-		(pts
 			(xy 207.01 90.17) (xy 209.55 90.17)
 		)
@@
 	(wire
 		(pts
-			(xy 86.36 48.26) (xy 99.06 48.26)
+			(xy 86.36 48.26) (xy 97.79 48.26)
 		)
 		(stroke
@@
 	(wire
 		(pts
-			(xy 100.33 48.26) (xy 102.87 48.26)
+			(xy 97.79 38.1) (xy 171.45 38.1)
 		)
 		(stroke
@@
 	(wire
 		(pts
-			(xy 99.06 38.1) (xy 171.45 38.1)
+			(xy 96.52 55.88) (xy 96.52 57.15)
 		)
 		(stroke
@@
 	(wire
 		(pts
-			(xy 96.52 55.88) (xy 96.52 57.15)
+			(xy 151.13 55.88) (xy 151.13 57.15)
 		)
 		(stroke
@@
 	(wire
 		(pts
-			(xy 151.13 55.88) (xy 151.13 57.15)
+			(xy 97.79 31.75) (xy 97.79 38.1)
 		)
 		(stroke
@@
 	(wire
 		(pts
-			(xy 99.06 48.26) (xy 99.06 38.1)
+			(xy 97.79 48.26) (xy 97.79 38.1)
 		)
 		(stroke
@@
 	(wire
 		(pts
+			(xy 97.79 48.26) (xy 102.87 48.26)
+		)
+		(stroke
+			(width 0)
+			(type default)
+		)
+	)
+	(wire
+		(pts
 			(xy 201.93 63.5) (xy 209.55 63.5)
 		)
@@
 	(symbol
 		(lib_id "Connector:TestPoint")
-		(at 100.33 66.04 180)
+		(at 97.79 31.75 0)
 		(unit 1)
 		(exclude_from_sim no)
@@
 		(fields_autoplaced yes)
 		(property "Reference" "SOLB1"
-			(at 102.87 68.0719 0)
+			(at 100.33 27.1779 0)
 			(effects
 				(font
 					(size 1.27 1.27)
 				)
-				(justify right)
+				(justify left)
 			)
 		)
 		(property "Value" "TestPoint"
-			(at 102.87 70.6119 0)
+			(at 100.33 29.7179 0)
 			(effects
 				(font
 					(size 1.27 1.27)
 				)
-				(justify right)
+				(justify left)
 			)
 		)
 		(property "Footprint" "TestPoint:TestPoint_Pad_1.0x1.0mm"
-			(at 95.25 66.04 0)
+			(at 102.87 31.75 0)
 			(effects
 				(font
@@
 		)
 		(property "Datasheet" "~"
-			(at 95.25 66.04 0)
+			(at 102.87 31.75 0)
 			(effects
 				(font
@@
 		)
 		(property "Description" "test point"
-			(at 100.33 66.04 0)
+			(at 97.79 31.75 0)
 			(effects
 				(font
