File: Plant_Saver_Spring_2026/Plant_Saver_Kicad_V2/Plant_Saver_Kicad_V2.kicad_sch (KiCad schematic)
At the start: 44 parts, among them J1 SBH11-PBPC-D05-ST-BK, J2 SBH11-PBPC-D05-ST-BK, J3 Test, J4 SM04B-SRSS-TB, J5 SM04B-SRSS-TB, J6 Conn_01x02_Pin, J7 Conn_01x06_Socket, J8 S3B-PH-K-S, Q1 G09P02L, Q2 G09P02L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

Commit message: Organized Repo
Parts:
- removed J3: Test, Connector_PinHeader_2.54mm:PinHeader_1x02_P2.54mm_Vertical, symbol Connector:Conn_01x02_Socket
- removed SW2: 1101M2S3AQE2, 1101M2S3AQE2:SPDT-1101M2_CNK, symbol Switch:SW_Wuerth_450301014042
- removed U1, U2, U3, U4: CDBA140SL-HF, CDBA140SL_HF:CDBA-HF, symbol CDBA140SL_HF:CDBA140SL-HF
- removed U17: LM66100DCK, Package_TO_SOT_SMD:SOT-363_SC-70-6, symbol Power_Management:LM66100DCK
- added C6: 100nF, Capacitor_SMD:C_1206_3216Metric_Pad1.33x1.80mm_HandSolder, symbol Device:C
- added U1, U12, U2, U3: LM66100DCK, Package_TO_SOT_SMD:SOT-363_SC-70-6, symbol LM66100DCKR:LM66100DCK
- SC1, SC2, SC3, SC4: value Solar_Cell -> SM400K10L-ND
Connections:
- net GND: now also C6.2, U1.2 (GND), U1.5 (ST), U12.2 (GND), U12.5 (ST), U2.2 (GND), U2.5 (ST), U3.2 (GND), U3.5 (ST)
- net Power_And_Charging/Solar: now also C6.1, U1.3 (~{CE}), U1.6 (VOUT), U12.3 (~{CE}), U12.6 (VOUT), U2.3 (~{CE}), U2.6 (VOUT), U3.3 (~{CE}), U3.6 (VOUT)
- net Power_And_Charging/Vbus_USB: now also J2.1
- net Solar_Measurement_Dual/Vin1: now also U12.1 (VIN)
- net Solar_Measurement_Dual/Vin2: now also U2.1 (VIN)
- net Solar_Measurement_Dual/Vin3: now also U1.1 (VIN)
- net Solar_Measurement_Dual/Vin4: now also U3.1 (VIN)
- net Vbus: no longer J2.1
- net Interface Stripboard/3V3 renamed Interface Stripboard/USB
Other:
- sheet Interface Stripboard ports: added USB; removed 3V3
- note added: "Can't use these ideal diodes, they won't survive the OSV"
- note added: "PMPP - 5.58 V, 15.4 mA SCV - 16.4 mA OCV - 6.91 V"
- note added: "TODO: Solar Charging/Energy collection"
- note removed: "TODO: Replace Regulator Switching stuff Schottky diodes Solar Charging/Energy collection Charging Lights off USB and not off switch"
- note removed: "Use these instead of Schottkys? Do they even work in RCB mode?"
- moved on the sheet: Boot1, C1, C2, C3, C4, CLK1, DAT1, GND1, H1, H2, J1, J2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

Commit message: Minor cleanup, slight tweaks in V2
Parts:
- J8: value S3B-PH-K-S -> 25SH-B-03-TR; footprint Connector_JST:JST_PH_S3B-PH-K_1x03_P2.00mm_Horizontal -> Connector_PinSocket_2.54mm:PinSocket_1x03_P2.54mm_Horizontal
Other:
- note added: "2.54 mm XH-style cable"
- note removed: "A03KR03KR26E152B"
Changed lines of the file:
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@@
 		)
 	)
-	(text "A03KR03KR26E152B"
+	(text "2.54 mm XH-style cable"
 		(exclude_from_sim no)
 		(at 482.8174 134.8465 0)
@@
 			)
 		)
-		(property "Value" "S3B-PH-K-S"
+		(property "Value" "25SH-B-03-TR"
 			(at 482.6 143.51 90)
 			(effects
@@
 			)
 		)
-		(property "Footprint" "Connector_JST:JST_PH_S3B-PH-K_1x03_P2.00mm_Horizontal"
+		(property "Footprint" "Connector_PinSocket_2.54mm:PinSocket_1x03_P2.54mm_Horizontal"
 			(at 482.6 146.05 0)
 			(effects

Commit message: Added assets for readme
Parts:
- removed U1, U12, U2, U3: LM66100DCK, Package_TO_SOT_SMD:SOT-363_SC-70-6, symbol LM66100DCKR:LM66100DCK
- added D4, D5, D6, D7: CRS10I30C(TE85L,QM, symbol Device:D_Schottky
Connections:
- net Power_And_Charging/Solar: now also D4.1 (K), D5.1 (K), D6.1 (K), D7.1 (K)
- net Solar_Measurement_Dual/Vin1: now also D4.2 (A)
- net Solar_Measurement_Dual/Vin2: now also D5.2 (A)
- net Solar_Measurement_Dual/Vin3: now also D6.2 (A)
- net Solar_Measurement_Dual/Vin4: now also D7.2 (A)
Other:
- note removed: "Can't use these ideal diodes, they won't survive the OSV"
- moved on the sheet: SC1, SC2, SC3, SC4
